File: Fuente/Fuente.kicad_sch (KiCad schematic)
At the start: 19 parts, among them J1 Bornera_VIN, J2 Bornera_VOUT, J4 Bornera_POT, J5 LED, J6 Bornera_POT, U1 LM317_TO-220

Commit message: .
Parts:
- removed TP1: TP_VIN, TestPoint:TestPoint_Pad_1.0x1.0mm, symbol Connector:TestPoint
- removed TP2: TP_VOUT, TestPoint:TestPoint_Pad_1.0x1.0mm, symbol Connector:TestPoint
- removed TP3: TP_GND, TestPoint:TestPoint_Pad_1.0x1.0mm, symbol Connector:TestPoint
- added A1: Arduino_101_Shield, PCM_arduino-library:Arduino_101_Shield, symbol PCM_arduino-library:Arduino_101_Shield
- added C5, C6: 100nF, Capacitor_THT:C_Disc_D5.0mm_W2.5mm_P5.00mm, symbol Device:C
- added D5: D_Zener, Diode_THT:D_A-405_P10.16mm_Horizontal, symbol Device:D_Zener
- added D6: TVS, Diode_THT:D_DO-201AE_P12.70mm_Horizontal, symbol Diode:1N62xxA
- added F1: Polyfuse, symbol Device:Polyfuse
- added J3: OLED, Connector_PinHeader_2.54mm:PinHeader_1x04_P2.54mm_Horizontal, symbol Connector:Conn_01x04_Pin
- added R10: 100k, Resistor_THT:R_Axial_DIN0207_L6.3mm_D2.5mm_P7.62mm_Horizontal, symbol Device:R
- added R3, R6: 100, Resistor_THT:R_Axial_DIN0207_L6.3mm_D2.5mm_P7.62mm_Horizontal, symbol Device:R
- added R4: 330, Resistor_THT:R_Axial_DIN0207_L6.3mm_D2.5mm_P7.62mm_Horizontal, symbol Device:R
- added R5: 220, Resistor_THT:R_Axial_DIN0207_L6.3mm_D2.5mm_P7.62mm_Horizontal, symbol Device:R
- added R7: rshunt, Resistor_THT:R_Axial_DIN0207_L6.3mm_D2.5mm_P7.62mm_Horizontal, symbol Device:R
- added R8, R9: 10k, Resistor_THT:R_Axial_DIN0207_L6.3mm_D2.5mm_P7.62mm_Horizontal, symbol Device:R
- added U2: LM317_TO-220, Package_TO_SOT_THT:TO-220-3_Vertical, symbol Regulator_Linear:LM317_TO-220
- added U3: LM358, Package_DIP:DIP-8_W7.62mm_Socket_LongPads, symbol Amplifier_Operational:LM358
Connections:
- net GND: now also A1.GND1 (GND), A1.GND2 (GND), A1.GND3 (GND), C5.2, C6.2, D5.2 (A), D6.2 (A2), J3.1 (Pin_1), R4.2, R6.2, R7.2, R8.1, R9.2, U3.4 (V-); no longer J2.1 (Pin_1)
- net VIN: no longer names the net of C1.1, C2.1, D2.1 (K), D4.1 (K), J5.2 (Pin_2), U1.3 (VI)
- net VIN: now also C5.1, D6.1 (A1), U2.3 (VI)
- net VOUT: no longer names the net of C3.1, C4.1, R2.1, U1.2 (VO)
- net VOUT: now also F1.1; no longer J2.2 (Pin_2)
- new net: R3.2, R4.1, U2.1 (ADJ)
- new net: R10.1, R9.1, U3.2 (-)
- new net +5V: A1.5V1 (5V), J3.2 (Pin_2), U3.8 (V+)
- new net +shunt: J2.1 (Pin_1), R7.1, R8.2, U3.3 (+)
- new net SCL: A1.A5, J3.4 (Pin_4)
- new net SDA: A1.A4, J3.3 (Pin_3)
- new net corriente: A1.A1, R10.2, U3.1
- new net vinArduino: A1.VIN, C6.1, D5.1 (K), R3.1, U2.2 (VO)
- new net voltaje: A1.A0, R5.2, R6.1
- new net vout: F1.2, J2.2 (Pin_2), R5.1
Other:
- note added: "¿Está bien el TVS ahí?"
- note added: "¿Está bien el zener?"
- note added: "¿Qué modelo de Rshunt se usa?"
- moved on the sheet: C1, C2, C3, C4, D1, D2, D3, D4, J1, J2, J4, J5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

Commit message: .
Parts:
- removed D6: TVS, Diode_THT:D_DO-201AE_P12.70mm_Horizontal, symbol Diode:1N62xxA
- removed R10: 100k, Resistor_THT:R_Axial_DIN0207_L6.3mm_D2.5mm_P7.62mm_Horizontal, symbol Device:R
- removed R7: rshunt, Resistor_THT:R_Axial_DIN0207_L6.3mm_D2.5mm_P7.62mm_Horizontal, symbol Device:R
- removed R8, R9: 10k, Resistor_THT:R_Axial_DIN0207_L6.3mm_D2.5mm_P7.62mm_Horizontal, symbol Device:R
- removed U3: LM358, Package_DIP:DIP-8_W7.62mm_Socket_LongPads, symbol Amplifier_Operational:LM358
- added J7: Conn_01x03_Pin, Connector_PinHeader_2.54mm:PinHeader_1x03_P2.54mm_Horizontal, symbol Connector:Conn_01x03_Pin
Connections:
- net +shunt is gone; now on net GND: J2.1 (Pin_1)
- net +5V: now also J7.1 (Pin_1)
- net GND: now also J7.3 (Pin_3)
- net corriente: now also J7.2 (Pin_2)
- net ADJ: no longer names the net of J4.2 (Pin_2), R2.2, U1.1 (ADJ)
Other:
- note removed: "¿Está bien el TVS ahí?"
- note removed: "¿Está bien el zener?"
- note removed: "¿Qué modelo de Rshunt se usa?"

Commit message: pcb terminada
Parts:
- removed J5: LED, Connector_PinHeader_2.54mm:PinHeader_1x02_P2.54mm_Vertical, symbol Connector:Conn_01x02_Pin
- added D6: LED, LED_THT:LED_D5.0mm, symbol Device:LED
- F1: footprint (none) -> Capacitor_THT:C_Disc_D5.0mm_W2.5mm_P5.00mm
- J4, J6: footprint TerminalBlock:TerminalBlock_MaiXu_MX126-5.0-02P_1x02_P5.00mm -> Connector_PinHeader_2.54mm:PinHeader_1x02_P2.54mm_Horizontal
Connections:
- net +5V: now also J7.2 (Pin_2); no longer J7.1 (Pin_1)
- net GND: no longer A1.GND2 (GND), A1.GND3 (GND)
- net corriente: now also J7.1 (Pin_1); no longer J7.2 (Pin_2)
- net at R1.1: now also D6.1 (K)
- net at C1.1, C2.1, C5.1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: now also D6.2 (A)
