File: Fuente/Fuente.kicad_pcb (KiCad board)
At the start: 2 copper layers, 46.7 x 31.2 mm, 19 parts, among them J1 Bornera_VIN, J2 Bornera_VOUT, J4 Bornera_POT, J5 LED, J6 Bornera_POT, U1 LM317_TO-220

Commit message: pcb terminada
Parts:
- removed J5: LED, Connector_PinHeader_2.54mm:PinHeader_1x02_P2.54mm_Vertical
- removed TP1: TP_VIN, TestPoint:TestPoint_Pad_1.0x1.0mm
- removed TP2: TP_VOUT, TestPoint:TestPoint_Pad_1.0x1.0mm
- removed TP3: TP_GND, TestPoint:TestPoint_Pad_1.0x1.0mm
- added A1: Arduino_101_Shield, PCM_arduino-library:Arduino_101_Shield, F.Cu at (30.0, 70.6)
- added C5: 100nF, Capacitor_THT:C_Disc_D5.0mm_W2.5mm_P5.00mm, F.Cu at (55.1, 29.1)
- added C6: 100nF, Capacitor_THT:C_Disc_D5.0mm_W2.5mm_P5.00mm, F.Cu at (39.3, 24.3)
- added D5: D_Zener, Diode_THT:D_A-405_P10.16mm_Horizontal, F.Cu at (31.5, 68.6)
- added D6: LED, LED_THT:LED_D5.0mm, F.Cu at (53.5, 42.4)
- added F1: Polyfuse, Capacitor_THT:C_Disc_D5.0mm_W2.5mm_P5.00mm, F.Cu at (93.0, 31.7)
- added J3: OLED, Connector_PinHeader_2.54mm:PinHeader_1x04_P2.54mm_Horizontal, F.Cu at (54.1, 59.2)
- added J7: Conn_01x03_Pin, Connector_PinHeader_2.54mm:PinHeader_1x03_P2.54mm_Horizontal, F.Cu at (40.9, 59.2)
- added R3: 100, Resistor_THT:R_Axial_DIN0207_L6.3mm_D2.5mm_P7.62mm_Horizontal, F.Cu at (43.6, 31.2)
- added R4: 330, Resistor_THT:R_Axial_DIN0207_L6.3mm_D2.5mm_P7.62mm_Horizontal, F.Cu at (51.2, 35.0)
- added R5: 220, Resistor_THT:R_Axial_DIN0207_L6.3mm_D2.5mm_P7.62mm_Horizontal, F.Cu at (83.8, 41.2)
- added R6: 100, Resistor_THT:R_Axial_DIN0207_L6.3mm_D2.5mm_P7.62mm_Horizontal, F.Cu at (79.4, 48.8)
- added U2: LM317_TO-220, Package_TO_SOT_THT:TO-220-3_Vertical, F.Cu at (44.7, 26.7)
- J4, J6: footprint TerminalBlock:TerminalBlock_MaiXu_MX126-5.0-02P_1x02_P5.00mm -> Connector_PinHeader_2.54mm:PinHeader_1x02_P2.54mm_Horizontal
- moved J1 52.8 mm to (24.6, 49.5), turned to 90 degrees
- moved J2 49.8 mm to (93.3, 46.7), turned to 90 degrees
- moved J4 36.6 mm to (74.2, 39.9), turned to -90 degrees
- moved C3 33.9 mm to (83.7, 25.3)
- moved C1 29.8 mm to (51.2, 50.7), turned to 90 degrees
- moved J6 25.8 mm to (67.1, 40.1), turned to -90 degrees
- moved D3 25.5 mm to (35.0, 44.5), turned to 0 degrees
- moved D1 25.1 mm to (35.0, 49.0), turned to 0 degrees
- moved R1 24.5 mm to (60.1, 41.8)
- moved D2 24.3 mm to (45.2, 53.2), turned to 180 degrees
- moved D4 23.4 mm to (45.2, 39.9), turned to 180 degrees
- moved C4 22.0 mm to (77.2, 24.1)
- moved R2 13.9 mm to (72.4, 31.9)
- moved U1 11.2 mm to (66.3, 26.4)
- moved C2 5.50 mm to (61.1, 29.1), turned to 90 degrees
Connections:
- net ADJ renamed Net-(J4-Pin_2)
- net VIN renamed Net-(D2-K)
- C3 pad 1: VOUT -> Net-(U1-VO)
- C4 pad 1: VOUT -> Net-(U1-VO)
- J2 pad 2: VOUT -> vout
- R2 pad 1: VOUT -> Net-(U1-VO)
- U1 pad 2: VOUT -> Net-(U1-VO)
Routing:
- net vinArduino: track 0.00 -> 131.7 mm
- net GND: track 104.0 -> 231.5 mm
- net VOUT: track 64.7 -> 0.00 mm
- net SDA: track 0.00 -> 59.3 mm
- net voltaje: track 0.00 -> 58.5 mm
- net SCL: track 0.00 -> 54.5 mm
- net +5V: track 0.00 -> 52.1 mm
- net corriente: track 0.00 -> 50.1 mm
- net Net-(U1-VO): track 0.00 -> 38.1 mm
- net Net-(D2-K): track 32.8 -> 69.1 mm
- net vout: track 0.00 -> 14.7 mm
- net Net-(U2-ADJ): track 0.00 -> 12.2 mm
- net Net-(D3-K): track 24.1 -> 15.0 mm
- net Net-(D1-K): track 23.4 -> 14.9 mm
- net Net-(J4-Pin_2): track 15.3 -> 20.2 mm
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Other:
- board outline removed

Commit message: .
Routing:
- net Net-(U1-VO): track 38.1 -> 41.0 mm
- net GND: track 231.5 -> 234.3 mm
- net Net-(D2-K): track 69.1 -> 66.9 mm
- net SDA: track 59.3 -> 61.5 mm
- net vinArduino: track 131.7 -> 133.5 mm
- net Net-(U2-ADJ): track 12.2 -> 13.6 mm
- net voltaje: track 58.5 -> 59.8 mm
Other:
- board text added: "SF 2026"
